Commit message: spawnato un blocco vero

File: blocks_description/X2-Y2_Z2.urdf.xacro (robot description, xacro)
@@ -4,5 +4,5 @@
     <visual>
       <geometry>
-        <mesh filename="/home/utente/my_ws/src/ur5lego/blocks_description/meshes/X2-Y2_Z2.dae.dae"/>
+        <mesh filename="/home/utente/my_ws/src/ur5lego/blocks_description/meshes/X2-Y2_Z2.dae"/>
       </geometry>
       <material name="Red">
@@ -12,5 +12,5 @@
     <collision>
       <geometry>
-        <mesh filename="/home/utente/my_ws/src/ur5lego/blocks_description/meshes/X2-Y2_Z2.dae.dae"/>
+        <mesh filename="/home/utente/my_ws/src/ur5lego/blocks_description/meshes/X2-Y2_Z2.dae"/>
       </geometry>
     </collision>
@@ -18,5 +18,5 @@
       <mass value="3.7"/>
       <origin rpy="0 0 0" xyz="0.0 0.0 0.0"/>
-      <inertia ixx="0.0" ixy="0.0" ixz="0.0" iyy="0.0" iyz="0.0" izz="0.0"/>
+      <inertia ixx="0.010267495893" ixy="0.0" ixz="0.0" iyy="0.010267495893" iyz="0.0" izz="0.00666"/>
     </inertial>
   </link>
