Commit message: parametrizzati nomi dei blocchi per spawnarne >1

File: blocks_description/X1-Y1-Z2.urdf.xacro (robot description, xacro)
@@ -1,5 +1,5 @@
 <?xml version="1.0"?>
-<!--<xacro:arg name="block_name" default="block"/>-->
-<robot xmlns:xacro="http://wiki.ros.org/xacro" name="haha">
+<robot xmlns:xacro="http://www.ros.org/wiki/xacro" name="$(arg block_name)">
+  <xacro:arg name="block_name" default="block"/>
   <link name="block">
     <visual>

File: blocks_description/X1-Y2-Z1.urdf.xacro (robot description, xacro)
@@ -1,4 +1,5 @@
 <?xml version="1.0"?>
-<robot xmlns:xacro="http://wiki.ros.org/xacro" name="$(arg robot_namespace)">
+<robot xmlns:xacro="http://www.ros.org/wiki/xacro" name="$(arg block_name)">
+  <xacro:arg name="block_name" default="block"/>
   <link name="block">
     <visual>

File: blocks_description/X1-Y2-Z2-CHAMFER.urdf.xacro (robot description, xacro)
@@ -1,5 +1,5 @@
 <?xml version="1.0"?>
-<xacro:arg name="block_name" default="block"/>
-<robot xmlns:xacro="http://wiki.ros.org/xacro" name="$(arg block_name)">
+<robot xmlns:xacro="http://www.ros.org/wiki/xacro" name="$(arg block_name)">
+  <xacro:arg name="block_name" default="block"/>
   <link name="block">
     <visual>

File: blocks_description/X1-Y2-Z2-TWINFILLET.urdf.xacro (robot description, xacro)
@@ -1,9 +1,9 @@
 <?xml version="1.0"?>
-<xacro:arg name="block_name" default="block"/>
-<robot xmlns:xacro="http://wiki.ros.org/xacro" name="$(arg block_name)">
+<robot xmlns:xacro="http://www.ros.org/wiki/xacro" name="$(arg block_name)">
+  <xacro:arg name="block_name" default="block"/>
   <link name="block">
     <visual>
       <geometry>
-        <mesh filename="$(find ur5lego)/blocks_description/meshes/X1-Y2-Z2-TWINFILLE.dae"/>
+        <mesh filename="$(find ur5lego)/blocks_description/meshes/X1-Y2-Z2-TWINFILLET.dae"/>
       </geometry>
       <material name="Red">
@@ -13,5 +13,5 @@
     <collision>
       <geometry>
-        <mesh filename="$(find ur5lego)/blocks_description/meshes/X1-Y2-Z2-TWINFILLE.dae"/>
+        <mesh filename="$(find ur5lego)/blocks_description/meshes/X1-Y2-Z2-TWINFILLET.dae"/>
       </geometry>
     </collision>

File: blocks_description/X1-Y2-Z2.urdf.xacro (robot description, xacro)
@@ -1,5 +1,5 @@
 <?xml version="1.0"?>
-<xacro:arg name="block_name" default="block"/>
-<robot xmlns:xacro="http://wiki.ros.org/xacro" name="$(arg block_name)">
+<robot xmlns:xacro="http://www.ros.org/wiki/xacro" name="$(arg block_name)">
+  <xacro:arg name="block_name" default="block"/>
   <link name="block">
     <visual>

File: blocks_description/X1-Y3-Z2-FILLET.urdf.xacro (robot description, xacro)
@@ -1,5 +1,5 @@
 <?xml version="1.0"?>
-<xacro:arg name="block_name" default="block"/>
-<robot xmlns:xacro="http://wiki.ros.org/xacro" name="$(arg block_name)">
+<robot xmlns:xacro="http://www.ros.org/wiki/xacro" name="$(arg block_name)">
+  <xacro:arg name="block_name" default="block"/>
   <link name="block">
     <visual>

File: blocks_description/X1-Y3-Z2.urdf.xacro (robot description, xacro)
@@ -1,5 +1,5 @@
 <?xml version="1.0"?>
-<xacro:arg name="block_name" default="block"/>
-<robot xmlns:xacro="http://wiki.ros.org/xacro" name="$(arg block_name)">
+<robot xmlns:xacro="http://www.ros.org/wiki/xacro" name="$(arg block_name)">
+  <xacro:arg name="block_name" default="block"/>
   <link name="block">
     <visual>

File: blocks_description/X1-Y4-Z1.urdf.xacro (robot description, xacro)
@@ -1,5 +1,5 @@
 <?xml version="1.0"?>
-<xacro:arg name="block_name" default="block"/>
-<robot xmlns:xacro="http://wiki.ros.org/xacro" name="$(arg block_name)">
+<robot xmlns:xacro="http://www.ros.org/wiki/xacro" name="$(arg block_name)">
+  <xacro:arg name="block_name" default="block"/>
   <link name="block">
     <visual>

File: blocks_description/X1-Y4-Z2.urdf.xacro (robot description, xacro)
@@ -1,5 +1,5 @@
 <?xml version="1.0"?>
-<xacro:arg name="block_name" default="block"/>
-<robot xmlns:xacro="http://wiki.ros.org/xacro" name="$(arg block_name)">
+<robot xmlns:xacro="http://www.ros.org/wiki/xacro" name="$(arg block_name)">
+  <xacro:arg name="block_name" default="block"/>
   <link name="block">
     <visual>

File: blocks_description/X2-Y2-Z2-FILLET.urdf.xacro (robot description, xacro)
@@ -1,5 +1,5 @@
 <?xml version="1.0"?>
-<xacro:arg name="block_name" default="block"/>
-<robot xmlns:xacro="http://wiki.ros.org/xacro" name="$(arg block_name)">
+<robot xmlns:xacro="http://www.ros.org/wiki/xacro" name="$(arg block_name)">
+  <xacro:arg name="block_name" default="block"/>
   <link name="block">
     <visual>

File: blocks_description/X2-Y2-Z2.urdf.xacro (robot description, xacro)
@@ -1,5 +1,5 @@
 <?xml version="1.0"?>
-<xacro:arg name="block_name" default="block"/>
-<robot xmlns:xacro="http://wiki.ros.org/xacro" name="$(arg block_name)">
+<robot xmlns:xacro="http://www.ros.org/wiki/xacro" name="$(arg block_name)">
+  <xacro:arg name="block_name" default="block"/>
   <link name="block">
     <visual>
