Commit message: added detection model

File: blocks_description/X1-Y2-Z2.urdf.xacro (robot description, xacro)
@@ -1,3 +1,4 @@
 <?xml version="1.0"?>
+<xacro:include filename="$(find ur5lego)/blocks_description/material.xacro" />
 <robot xmlns:xacro="http://www.ros.org/wiki/xacro" name="$(arg block_name)">
   <xacro:arg name="block_name" default="block"/>
@@ -7,7 +8,5 @@
         <mesh filename="$(find ur5lego)/blocks_description/meshes/X1-Y2-Z2.dae"/>
       </geometry>
-      <material name="Red">
-        <color rgba="1.0 0.0 0.0 1.0"/>
-      </material>
+      <material name="random_color"/>
     </visual>
     <collision>

File: blocks_description/X1-Y4-Z2.urdf.xacro (robot description, xacro)
@@ -2,4 +2,7 @@
 <robot xmlns:xacro="http://www.ros.org/wiki/xacro" name="$(arg block_name)">
   <xacro:arg name="block_name" default="block"/>
+  <material name="Orange">
+    <color rgba="${255/255} ${108/255} ${10/255} 1.0"/>
+  </material>
   <link name="block">
     <visual>
@@ -7,7 +10,5 @@
         <mesh filename="$(find ur5lego)/blocks_description/meshes/X1-Y4-Z2.dae"/>
       </geometry>
-      <material name="Red">
-        <color rgba="1.0 0.0 0.0 1.0"/>
-      </material>
+      <material name="Orange"/>
     </visual>
     <collision>
@@ -22,3 +23,6 @@
     </inertial>
   </link>
+  <gazebo reference="block">
+    <material>Gazebo/Blue</material>
+  </gazebo>
 </robot>
