Commit message: pulito codice

File: robot_description/ur5.urdf.xacro (robot description, xacro)
@@ -6,4 +6,9 @@
 <xacro:arg name="gripper" default="false"/>
 <xacro:arg name="prefix" default=""/>
+<!-- legal values:
+ - hardware_interface/PositionJointInterface
+ - hardware_interface/VelocityJointInterface
+ - hardware_interface/EffortJointInterface
+-->
 <xacro:arg name="transmission_hw_interface" default="hardware_interface/EffortJointInterface"/>
 <xacro:arg name="joint_limit_params" default="config/joint_limits.yaml"/>
@@ -11,9 +16,4 @@
 <xacro:arg name="physical_params" default="config/physical_parameters.yaml"/>
 <xacro:arg name="visual_params" default="config/visual_parameters.yaml"/>
-<!-- legal values:
- - hardware_interface/PositionJointInterface
- - hardware_interface/VelocityJointInterface
- - hardware_interface/EffortJointInterface
--->
 <xacro:arg name="safety_limits" default="false"/>
 <xacro:arg name="safety_pos_margin" default="0.15"/>
@@ -57,9 +57,9 @@
 		<origin xyz="0.05 0.0 -0.02" rpy="0 -1.57 0.0"/>
 	</xacro:d435_camera>
-	  <xacro:property name="camera_fov" value="3.0"/>
-	  <xacro:property name="camera_width" value="640"/>
-	  <xacro:property name="camera_height" value="480"/>
-	  <xacro:property name="camera_near" value="0.01"/>
-	  <xacro:property name="camera_far" value="100"/>
+	<xacro:property name="camera_fov" value="3.0"/>
+	<xacro:property name="camera_width" value="640"/>
+	<xacro:property name="camera_height" value="480"/>
+	<xacro:property name="camera_near" value="0.01"/>
+	<xacro:property name="camera_far" value="100"/>
 	<xacro:d435_camera
 		parent="base_link"
@@ -70,11 +70,4 @@
 </xacro:if>
 <xacro:if value="$(arg gazebo)">
-  <!--
-    Attach the Gazebo model to Gazebo's world frame.
-    Note: if you're looking to integrate a UR into a larger scene and need
-    to add EEFs or other parts, DO NOT change this file or the 'world' link
-    here. Create a NEW xacro instead and decide whether you need to add
-    a 'world' link there.
-  -->
   <link name="world"/>
   <joint name="world_joint" type="fixed">
@@ -132,5 +125,5 @@
     <gazebo>
       <plugin name="gazebo_ros_controller_manager" filename="libgazebo_ros_control.so">
-			<robotNamespace>/ur5</robotNamespace> <!--TODO1 change this with prefix when you use 2 robots     -->
+			<robotNamespace>/ur5</robotNamespace>
 			<robotSimType>gazebo_ros_control/DefaultRobotHWSim</robotSimType>
 			<legacyModeNS>true</legacyModeNS>

Commit message: zed_camera giusta

File: robot_description/ur5.urdf.xacro (robot description, xacro)
@@ -41,14 +41,24 @@
 </joint>
 <xacro:if value="$(arg vision_sensor)">
-	<xacro:include filename="sensors/d435_camera.urdf.xacro"/>
+	<xacro:if value="$(arg gazebo)">
+		<xacro:include filename="sensors/zed2/simulation/zed2.xacro"/>
+		<xacro:zed2
+			parent="base_link"
+			name="zed_camera1">
+			<origin xyz="-0.9 0.18 -0.35" rpy="0. 0.523 0."/>
+		</xacro:zed2>
+		<xacro:zed2_gazebo/>
+  	</xacro:if>
+	<!-- <xacro:include filename="sensors/d435_camera.urdf.xacro"/>-->
 	  <!-- realsense -->
 	  <!--These values are taken from  d435_camera.urdf.xacro and  d435_camera_openni.gazebo.urdf.xacro in sensors-description
 	 repo, commit 3fb6f787-->
-	  <xacro:property name="camera_fov" value="3.0"/>
+	<!--
+	  <xacro:property name="camera_fov" value="1.0"/>
 	  <xacro:property name="camera_width" value="640"/>
 	  <xacro:property name="camera_height" value="480"/>
 	  <xacro:property name="camera_near" value="0.1"/>
 	  <xacro:property name="camera_far" value="100"/>
-	  <xacro:property name="m_camera" value="0.07"/> <!--??-->
+	  <xacro:property name="m_camera" value="0.07"/>
 	<xacro:d435_camera
 		parent="wrist_3_link"
@@ -57,5 +67,5 @@
 		<origin xyz="0.05 0.0 -0.02" rpy="0 -1.57 0.0"/>
 	</xacro:d435_camera>
-	<xacro:property name="camera_fov" value="3.0"/>
+	<xacro:property name="camera_fov" value="1.0"/>
 	<xacro:property name="camera_width" value="640"/>
 	<xacro:property name="camera_height" value="480"/>
@@ -67,5 +77,5 @@
 		camera_plugin="true">
 		<origin xyz="0.0 -0.3 -0.5" rpy="0.0  0.5 1.57"/>
-	</xacro:d435_camera>
+	</xacro:d435_camera> -->
 </xacro:if>
 <xacro:if value="$(arg gazebo)">
