Commit message: cambiato l'urdf così a caso

File: robot_description/ur5.urdf (robot description, URDF)
Before this commit: robot ur5, 41 links, 40 joints
Links:
- removed link base_link_inertia
- removed link ee_camera/camera_bottom_screw_frame
- removed link ee_camera/camera_color_frame
- removed link ee_camera/camera_color_optical_frame
- removed link ee_camera/camera_depth_frame
- removed link ee_camera/camera_depth_optical_frame
- removed link ee_camera/camera_left_ir_frame
- removed link ee_camera/camera_left_ir_optical_frame
- removed link ee_camera/camera_link
- removed link ee_camera/camera_right_ir_frame
- removed link ee_camera/camera_right_ir_optical_frame
- removed link flange
- removed link forearm_link_end
- removed link forearm_link_middle
- removed link gripper_base
- removed link gripper_base_down
- removed link hand_1_link
- removed link hand_2_link
- removed link hand_3_link
- removed link tool0_without_gripper
- removed link upper_arm_link_middle
- removed link z_base_camera/camera_bottom_screw_frame
- removed link z_base_camera/camera_color_frame
- removed link z_base_camera/camera_color_optical_frame
- removed link z_base_camera/camera_depth_frame
- removed link z_base_camera/camera_depth_optical_frame
- removed link z_base_camera/camera_left_ir_frame
- removed link z_base_camera/camera_left_ir_optical_frame
- removed link z_base_camera/camera_link
- removed link z_base_camera/camera_right_ir_frame
- removed link z_base_camera/camera_right_ir_optical_frame
- added link ee_link; collision box size=0.01 0.01 0.01
- link base_link: mass None -> 4.0; geometry collision mesh filename=package://example-robot-data/robots/ur_description/meshes/u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; visual mesh filename=package://example-robot-data/robots/ur_description/meshes/u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
- link forearm_link: geometry collision mesh filename=package://example-robot-data/robots/ur_description/meshes/u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; visual mesh filename=package://example-robot-data/robots/ur_description/meshes/u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
- link shoulder_link: geometry collision mesh filename=package://example-robot-data/robots/ur_description/meshes/u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; visual mesh filename=package://example-robot-data/robots/ur_description/meshes/u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
- link tool0: geometry collision box size=0.005 0.02 0.05; collision box size=0.005 0.02 0.05
- link upper_arm_link: geometry collision mesh filename=package://example-robot-data/robots/ur_description/meshes/u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; visual mesh filename=package://example-robot-data/robots/ur_description/meshes/u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
- link wrist_1_link: geometry collision mesh filename=package://example-robot-data/robots/ur_description/meshes/u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; visual mesh filename=package://example-robot-data/robots/ur_description/meshes/u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
- link wrist_2_link: geometry collision mesh filename=package://example-robot-data/robots/ur_description/meshes/u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; visual mesh filename=package://example-robot-data/robots/ur_description/meshes/u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
- link wrist_3_link: geometry collision mesh filename=package://example-robot-data/robots/ur_description/meshes/u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; visual mesh filename=package://example-robot-data/robots/ur_description/meshes/u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
Joints:
- removed joint base_link-base_link_inertia
- removed joint ee_camera/camera_color_joint
- removed joint ee_camera/camera_color_optical_joint
- removed joint ee_camera/camera_depth_joint
- removed joint ee_camera/camera_depth_optical_joint
- removed joint ee_camera/camera_left_ir_joint
- removed joint ee_camera/camera_left_ir_optical_joint
- removed joint ee_camera/camera_link_joint
- removed joint ee_camera/camera_right_ir_joint
- removed joint ee_camera/camera_right_ir_optical_joint
- removed joint ee_camera/wrist_3_linkcamera_joint
- removed joint fixed_ee_gripper
- removed joint flange
- removed joint flange-tool0
- removed joint forearm_link_end_fixed_joint
- removed joint forearm_link_middle_fixed_joint
- removed joint gripper_robot_joint
- removed joint hand_1_joint
- removed joint hand_2_joint
- removed joint hand_3_joint
- removed joint upper_arm_link_middle_fixed_joint
- removed joint wrist_3-flange
- removed joint z_base_camera/base_linkcamera_joint
- removed joint z_base_camera/camera_color_joint
- removed joint z_base_camera/camera_color_optical_joint
- removed joint z_base_camera/camera_depth_joint
- removed joint z_base_camera/camera_depth_optical_joint
- removed joint z_base_camera/camera_left_ir_joint
- removed joint z_base_camera/camera_left_ir_optical_joint
- removed joint z_base_camera/camera_link_joint
- removed joint z_base_camera/camera_right_ir_joint
- removed joint z_base_camera/camera_right_ir_optical_joint
- added joint ee_fixed_joint: type fixed, parent wrist_3_link, child ee_link, origin xyz=0.0 0.0823 0.0 rpy=0.0 0.0 1.570796325
- added joint wrist_3_link-tool0_fixed_joint: type fixed, parent wrist_3_link, child tool0, origin xyz=0 0.0823 0 rpy=-1.570796325 0 0
- joint base_link-base_fixed_joint: origin xyz=0 0 0 rpy=0 0 3.141592653589793 -> xyz=0 0 0 rpy=0 0 -3.14159265
- joint elbow_joint: axis 0 0 1 -> 0 1 0; limit lower=-3.14 upper=3.14 effort=150.0 velocity=3.14 -> lower=-3.14159265 upper=3.14159265 effort=150.0 velocity=3.15; origin xyz=-0.425 0 0 rpy=0 0 0 -> xyz=0.0 -0.1197 0.425 rpy=0.0 0.0 0.0
- joint shoulder_lift_joint: axis 0 0 1 -> 0 1 0; limit lower=-3.14 upper=0 effort=150.0 velocity=3.14 -> lower=-3.14159265 upper=3.14159265 effort=150.0 velocity=3.15; origin xyz=0 0 0 rpy=1.570796327 0 0 -> xyz=0.0 0.13585 0.0 rpy=0.0 1.570796325 0.0
- joint shoulder_pan_joint: limit lower=-6.14 upper=6.14 effort=150.0 velocity=3.14 -> lower=-3.14159265 upper=3.14159265 effort=150.0 velocity=3.15; origin xyz=0 0 0.1625 rpy=0 0 0 -> xyz=0.0 0.0 0.089159 rpy=0.0 0.0 0.0; parent base_link_inertia -> base_link
- joint world_joint: origin xyz=0 0 0 rpy=0 0 0 -> xyz=0.0 0.0 0.0 rpy=0.0 0.0 0.0
- joint wrist_1_joint: axis 0 0 1 -> 0 1 0; limit lower=-6.28 upper=6.28 effort=28.0 velocity=3.14 -> lower=-3.14159265 upper=3.14159265 effort=28.0 velocity=3.2; origin xyz=-0.3922 0 0.1333 rpy=0 0 0 -> xyz=0.0 0.0 0.39225 rpy=0.0 1.570796325 0.0
- joint wrist_2_joint: limit lower=-6.28 upper=6.28 effort=28.0 velocity=3.14 -> lower=-3.14159265 upper=3.14159265 effort=28.0 velocity=3.2; origin xyz=0 -0.0997 -2.044881182297852e-11 rpy=1.570796327 0 0 -> xyz=0.0 0.093 0.0 rpy=0.0 0.0 0.0
- joint wrist_3_joint: axis 0 0 1 -> 0 1 0; limit lower=-6.28 upper=6.28 effort=28.0 velocity=3.14 -> lower=-3.14159265 upper=3.14159265 effort=28.0 velocity=3.2; origin xyz=0 0.0996 -2.042830148012698e-11 rpy=1.570796326589793 3.141592653589793 3.141592653589793 -> xyz=0.0 0.0 0.09465 rpy=0.0 0.0 0.0

Commit message: inserito joint gripper

File: robot_description/ur5.urdf (robot description, URDF)
Before this commit: robot ur5, 11 links, 10 joints
Links:
- removed link ee_link
- added link base_link_inertia, mass 4.0; collision mesh filename=package://ur_description/meshes/ur5e/collision/base.stl; visual mesh filename=package://ur_description/meshes/ur5e/visual/base.dae
- added link flange
- added link forearm_link_end
- added link forearm_link_middle
- added link gripper_base; collision mesh filename=package://gripper_description/meshes/gripper_base_up.stl scale=0.001 0.001 0.001; visual mesh filename=package://gripper_description/meshes/gripper_base_up.stl scale=0.001 0.001 0.001
- added link gripper_base_down, mass 1.0; collision mesh filename=package://gripper_description/meshes/gripper_base_down.stl scale=0.001 0.001 0.001; visual mesh filename=package://gripper_description/meshes/gripper_base_down.stl scale=0.001 0.001 0.001
- added link hand_1_link, mass 0.05; collision mesh filename=package://gripper_description/meshes/finger.stl scale=0.001 0.001 0.001; visual mesh filename=package://gripper_description/meshes/finger.stl scale=0.001 0.001 0.001
- added link hand_2_link, mass 0.05; collision mesh filename=package://gripper_description/meshes/finger.stl scale=0.001 0.001 0.001; visual mesh filename=package://gripper_description/meshes/finger.stl scale=0.001 0.001 0.001
- added link hand_3_link, mass 0.05; collision mesh filename=package://gripper_description/meshes/finger.stl scale=0.001 0.001 0.001; visual mesh filename=package://gripper_description/meshes/finger.stl scale=0.001 0.001 0.001
- added link tool0_without_gripper
- added link upper_arm_link_middle
- added link zed2_baro_link
- added link zed2_camera_center, mass 0.16140; collision mesh filename=package://ur_description/sensors/zed2/simulation/ZED2.dae; visual mesh filename=package://ur_description/sensors/zed2/simulation/ZED2.dae
- added link zed2_left_camera_frame
- added link zed2_left_camera_optical_frame
- added link zed2_mag_link
- added link zed2_right_camera_frame
- added link zed2_right_camera_optical_frame
- added link zed2_temp_left_link
- added link zed2_temp_right_link
- link base_link: mass 4.0 -> None; geometry 
- link forearm_link: geometry collision mesh filename=package://ur_description/meshes/ur5e/collision/forearm.stl; visual mesh filename=package://ur_description/meshes/ur5e/visual/forearm.dae
- link shoulder_link: geometry collision mesh filename=package://ur_description/meshes/ur5e/collision/shoulder.stl; visual mesh filename=package://ur_description/meshes/ur5e/visual/shoulder.dae
- link tool0: geometry 
- link upper_arm_link: geometry collision mesh filename=package://ur_description/meshes/ur5e/collision/upperarm.stl; visual mesh filename=package://ur_description/meshes/ur5e/visual/upperarm.dae
- link wrist_1_link: geometry collision mesh filename=package://ur_description/meshes/ur5e/collision/wrist1.stl; visual mesh filename=package://ur_description/meshes/ur5e/visual/wrist1.dae
- link wrist_2_link: geometry collision mesh filename=package://ur_description/meshes/ur5e/collision/wrist2.stl; visual mesh filename=package://ur_description/meshes/ur5e/visual/wrist2.dae
- link wrist_3_link: geometry collision mesh filename=package://ur_description/meshes/ur5e/collision/wrist3.stl; visual mesh filename=package://ur_description/meshes/ur5e/visual/wrist3.dae
Joints:
- removed joint ee_fixed_joint
- removed joint wrist_3_link-tool0_fixed_joint
- added joint base_link-base_link_inertia: type fixed, parent base_link, child base_link_inertia, origin xyz=0 0 0 rpy=3.141592653589793 0 0
- added joint fixed_ee_gripper: type fixed, parent gripper_base, child tool0, origin xyz=0 0 0.12 rpy=0 0 0
- added joint flange: type fixed, parent gripper_base, child gripper_base_down, origin xyz=0 0 0.06 rpy=0 0 0
- added joint flange-tool0: type fixed, parent flange, child tool0_without_gripper, origin xyz=0 0 0 rpy=1.5707963267948966 0 1.5707963267948966
- added joint forearm_link_end_fixed_joint: type fixed, parent forearm_link, child forearm_link_end, origin xyz=-0.425 0 0 rpy=0 0 0
- added joint forearm_link_middle_fixed_joint: type fixed, parent forearm_link, child forearm_link_middle, origin xyz=-0.2125 0.0 0.0 rpy=0 0 0
- added joint gripper_robot_joint: type fixed, parent tool0_without_gripper, child gripper_base, origin xyz=0 0 0 rpy=0 0 1.57
- added joint hand_1_joint: type fixed, parent gripper_base_down, child hand_1_link, origin xyz=0.0  -0.03 0.05 rpy=-1.5707963267948966 0 0
- added joint hand_2_joint: type fixed, parent gripper_base_down, child hand_2_link, origin xyz=0.02598 0.015 0.05 rpy=-1.5707963267948966 0 2.0943951023931953
- added joint hand_3_joint: type fixed, parent gripper_base_down, child hand_3_link, origin xyz=-0.02598 0.015 0.05 rpy=-1.5707963267948966 0 -2.0943951023931953
- added joint upper_arm_link_middle_fixed_joint: type fixed, parent upper_arm_link, child upper_arm_link_middle, origin xyz=-0.2125 0 0.13 rpy=0 0 0
- added joint wrist_3-flange: type fixed, parent wrist_3_link, child flange, origin xyz=0 0 0 rpy=0 -1.5707963267948966 -1.5707963267948966
- added joint zed2_baro_joint: type fixed, parent zed2_camera_center, child zed2_baro_link, origin xyz=0 0 0 rpy=0 0 0
- added joint zed2_left_camera_joint: type fixed, parent zed2_camera_center, child zed2_left_camera_frame, origin xyz=0 0.06 0 rpy=0 0 0
- added joint zed2_left_camera_optical_joint: type fixed, parent zed2_left_camera_frame, child zed2_left_camera_optical_frame, origin xyz=0 0 0 rpy=-1.5707963267948966 0.0 -1.5707963267948966
- added joint zed2_mag_joint: type fixed, parent zed2_camera_center, child zed2_mag_link, origin xyz=0 0 0 rpy=0 0 0
- added joint zed2_right_camera_joint: type fixed, parent zed2_camera_center, child zed2_right_camera_frame, origin xyz=0 -0.06 0 rpy=0 0 0
- added joint zed2_right_camera_optical_joint: type fixed, parent zed2_right_camera_frame, child zed2_right_camera_optical_frame, origin xyz=0 0 0 rpy=-1.5707963267948966 0.0 -1.5707963267948966
- added joint zed2_temp_left_joint: type fixed, parent zed2_left_camera_frame, child zed2_temp_left_link, origin xyz=0 0 0 rpy=0 0 0
- added joint zed2_temp_right_joint: type fixed, parent zed2_right_camera_frame, child zed2_temp_right_link, origin xyz=0 0 0 rpy=0 0 0
- added joint zed_camera_fixed_joint: type fixed, parent base_link, child zed2_camera_center, origin xyz=-0.9 0.18 -0.35 rpy=0. 0.523 0.
- joint base_link-base_fixed_joint: origin xyz=0 0 0 rpy=0 0 -3.14159265 -> xyz=0 0 0 rpy=0 0 3.141592653589793
- joint elbow_joint: axis 0 1 0 -> 0 0 1; limit lower=-3.14159265 upper=3.14159265 effort=150.0 velocity=3.15 -> lower=-3.14 upper=3.14 effort=150.0 velocity=3.14; origin xyz=0.0 -0.1197 0.425 rpy=0.0 0.0 0.0 -> xyz=-0.425 0 0 rpy=0 0 0
- joint shoulder_lift_joint: axis 0 1 0 -> 0 0 1; limit lower=-3.14159265 upper=3.14159265 effort=150.0 velocity=3.15 -> lower=-3.14 upper=0 effort=150.0 velocity=3.14; origin xyz=0.0 0.13585 0.0 rpy=0.0 1.570796325 0.0 -> xyz=0 0 0 rpy=1.570796327 0 0
- joint shoulder_pan_joint: limit lower=-3.14159265 upper=3.14159265 effort=150.0 velocity=3.15 -> lower=-6.14 upper=6.14 effort=150.0 velocity=3.14; origin xyz=0.0 0.0 0.089159 rpy=0.0 0.0 0.0 -> xyz=0 0 0.1625 rpy=0 0 0; parent base_link -> base_link_inertia
- joint world_joint: origin xyz=0.0 0.0 0.0 rpy=0.0 0.0 0.0 -> xyz=0 0 0 rpy=0 0 0
- joint wrist_1_joint: axis 0 1 0 -> 0 0 1; limit lower=-3.14159265 upper=3.14159265 effort=28.0 velocity=3.2 -> lower=-6.28 upper=6.28 effort=28.0 velocity=3.14; origin xyz=0.0 0.0 0.39225 rpy=0.0 1.570796325 0.0 -> xyz=-0.3922 0 0.1333 rpy=0 0 0
- joint wrist_2_joint: limit lower=-3.14159265 upper=3.14159265 effort=28.0 velocity=3.2 -> lower=-6.28 upper=6.28 effort=28.0 velocity=3.14; origin xyz=0.0 0.093 0.0 rpy=0.0 0.0 0.0 -> xyz=0 -0.0997 -2.044881182297852e-11 rpy=1.570796327 0 0
- joint wrist_3_joint: axis 0 1 0 -> 0 0 1; limit lower=-3.14159265 upper=3.14159265 effort=28.0 velocity=3.2 -> lower=-6.28 upper=6.28 effort=28.0 velocity=3.14; origin xyz=0.0 0.0 0.09465 rpy=0.0 0.0 0.0 -> xyz=0 0.0996 -2.042830148012698e-11 rpy=1.570796326589793 3.141592653589793 3.141592653589793

File: robot_description/ur5.urdf.xacro (robot description, xacro)
@@ -4,5 +4,5 @@
 <xacro:arg name="vision_sensor" default="true"/>
 <xacro:arg name="gazebo" default="true"/>
-<xacro:arg name="gripper" default="false"/>
+<xacro:arg name="gripper" default="true"/>
 <xacro:arg name="prefix" default=""/>
 <!-- legal values:

Commit message: funziona

File: robot_description/ur5.urdf (robot description, URDF)
Before this commit: robot ur_robot, 30 links, 29 joints
Links:
- removed link base_link_inertia
- removed link flange
- removed link forearm_link_end
- removed link forearm_link_middle
- removed link gripper_base
- removed link gripper_base_down
- removed link hand_1_link
- removed link hand_2_link
- removed link hand_3_link
- removed link tool0_without_gripper
- removed link upper_arm_link_middle
- removed link zed2_baro_link
- removed link zed2_camera_center
- removed link zed2_left_camera_frame
- removed link zed2_left_camera_optical_frame
- removed link zed2_mag_link
- removed link zed2_right_camera_frame
- removed link zed2_right_camera_optical_frame
- removed link zed2_temp_left_link
- removed link zed2_temp_right_link
- added link ee_link; collision box size=0.01 0.01 0.01
- link base_link: mass None -> 4.0; geometry collision mesh filename=package://example-robot-data/robots/ur_description/meshes/u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; visual mesh filename=package://example-robot-data/robots/ur_description/meshes/u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
- link forearm_link: geometry collision mesh filename=package://example-robot-data/robots/ur_description/meshes/u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; visual mesh filename=package://example-robot-data/robots/ur_description/meshes/u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
- link shoulder_link: geometry collision mesh filename=package://example-robot-data/robots/ur_description/meshes/u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; visual mesh filename=package://example-robot-data/robots/ur_description/meshes/u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
- link tool0: geometry collision box size=0.005 0.02 0.05; collision box size=0.005 0.02 0.05
- link upper_arm_link: geometry collision mesh filename=package://example-robot-data/robots/ur_description/meshes/u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; visual mesh filename=package://example-robot-data/robots/ur_description/meshes/u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
- link wrist_1_link: geometry collision mesh filename=package://example-robot-data/robots/ur_description/meshes/u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; visual mesh filename=package://example-robot-data/robots/ur_description/meshes/u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
- link wrist_2_link: geometry collision mesh filename=package://example-robot-data/robots/ur_description/meshes/u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; visual mesh filename=package://example-robot-data/robots/ur_description/meshes/u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
- link wrist_3_link: geometry collision mesh filename=package://example-robot-data/robots/ur_description/meshes/u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; visual mesh filename=package://example-robot-data/robots/ur_description/meshes/u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
Joints:
- removed joint base_link-base_link_inertia
- removed joint fixed_ee_gripper
- removed joint flange
- removed joint flange-tool0
- removed joint forearm_link_end_fixed_joint
- removed joint forearm_link_middle_fixed_joint
- removed joint gripper_robot_joint
- removed joint hand_1_joint
- removed joint hand_2_joint
- removed joint hand_3_joint
- removed joint upper_arm_link_middle_fixed_joint
- removed joint wrist_3-flange
- removed joint zed2_baro_joint
- removed joint zed2_left_camera_joint
- removed joint zed2_left_camera_optical_joint
- removed joint zed2_mag_joint
- removed joint zed2_right_camera_joint
- removed joint zed2_right_camera_optical_joint
- removed joint zed2_temp_left_joint
- removed joint zed2_temp_right_joint
- removed joint zed_camera_fixed_joint
- added joint ee_fixed_joint: type fixed, parent wrist_3_link, child ee_link, origin xyz=0.0 0.0823 0.0 rpy=0.0 0.0 1.570796325
- added joint wrist_3_link-tool0_fixed_joint: type fixed, parent wrist_3_link, child tool0, origin xyz=0 0.0823 0 rpy=-1.570796325 0 0
- joint base_link-base_fixed_joint: origin xyz=0 0 0 rpy=0 0 3.141592653589793 -> xyz=0 0 0 rpy=0 0 -3.14159265
- joint elbow_joint: axis 0 0 1 -> 0 1 0; limit lower=-3.14 upper=3.14 effort=150.0 velocity=3.14 -> lower=-3.14159265 upper=3.14159265 effort=150.0 velocity=3.15; origin xyz=-0.425 0 0 rpy=0 0 0 -> xyz=0.0 -0.1197 0.425 rpy=0.0 0.0 0.0
- joint shoulder_lift_joint: axis 0 0 1 -> 0 1 0; limit lower=-3.14 upper=0 effort=150.0 velocity=3.14 -> lower=-3.14159265 upper=3.14159265 effort=150.0 velocity=3.15; origin xyz=0 0 0 rpy=1.570796327 0 0 -> xyz=0.0 0.13585 0.0 rpy=0.0 1.570796325 0.0
- joint shoulder_pan_joint: limit lower=-6.14 upper=6.14 effort=150.0 velocity=3.14 -> lower=-3.14159265 upper=3.14159265 effort=150.0 velocity=3.15; origin xyz=0 0 0.1625 rpy=0 0 0 -> xyz=0.0 0.0 0.089159 rpy=0.0 0.0 0.0; parent base_link_inertia -> base_link
- joint world_joint: origin xyz=0 0 0 rpy=0 0 0 -> xyz=0.0 0.0 0.0 rpy=0.0 0.0 0.0
- joint wrist_1_joint: axis 0 0 1 -> 0 1 0; limit lower=-6.28 upper=6.28 effort=28.0 velocity=3.14 -> lower=-3.14159265 upper=3.14159265 effort=28.0 velocity=3.2; origin xyz=-0.3922 0 0.1333 rpy=0 0 0 -> xyz=0.0 0.0 0.39225 rpy=0.0 1.570796325 0.0
- joint wrist_2_joint: limit lower=-6.28 upper=6.28 effort=28.0 velocity=3.14 -> lower=-3.14159265 upper=3.14159265 effort=28.0 velocity=3.2; origin xyz=0 -0.0997 -2.044881182297852e-11 rpy=1.570796327 0 0 -> xyz=0.0 0.093 0.0 rpy=0.0 0.0 0.0
- joint wrist_3_joint: axis 0 0 1 -> 0 1 0; limit lower=-6.28 upper=6.28 effort=28.0 velocity=3.14 -> lower=-3.14159265 upper=3.14159265 effort=28.0 velocity=3.2; origin xyz=0 0.0996 -2.042830148012698e-11 rpy=1.570796326589793 3.141592653589793 3.141592653589793 -> xyz=0.0 0.0 0.09465 rpy=0.0 0.0 0.0
